File: src/shift-register-control-panel.kicad_sch (KiCad schematic)
At the start: 34 parts, among them J1 Conn_01x08, J2 USB_A, SW1 INPUT, SW2 SHIFT, SW3 CLEAR, SW4 DISPLAY, U1 74HC595, U2 LM7805_TO220, U3 SN74LVC1G14

Commit message: updated with OSH Park DRC
Parts:
- removed C2: 100 nF, Capacitor_THT:C_Disc_D5.0mm_W2.5mm_P5.00mm, symbol Device:C
- removed J2: USB_A, Connector_USB:USB_A_Molex_67643_Horizontal, symbol Connector:USB_A
- removed U3: SN74LVC1G14, Package_TO_SOT_SMD:SOT-23-5, symbol 74xGxx:SN74LVC1G14DBV
- added J2: Conn_01x03, symbol Connector_Generic:Conn_01x03
- added U3: 74HC14, symbol 74xx:74HC14
- C3: footprint Capacitor_THT:C_Disc_D5.0mm_W2.5mm_P5.00mm -> (none)
- U2: value LM7805_TO220 -> LM7805
Connections:
- net +5V: now also C3.1, J2.2 (Pin_2), U3.14 (VCC); no longer C3.2
- net GND: now also C3.2, J2.3 (Pin_3), U3.7 (GND); no longer C3.1
- net VCC: now also J2.1 (Pin_1)
- net at C1.1, R10.2: now also U3.1
- net at U1.11 (SRCLK): now also U3.2
- no-connect marks 3 -> 11
Other:
- moved on the sheet: C1, D1, D2, D3, D4, D5, D6, D7, D8, D9, J1, R1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

Commit message: should have been part of last commit
Parts:
- C3: footprint (none) -> Capacitor_THT:C_Disc_D5.0mm_W2.5mm_P5.00mm
- J2: footprint (none) -> Connector_PinHeader_2.54mm:PinHeader_1x03_P2.54mm_Vertical
- U3: footprint (none) -> Package_DIP:DIP-14_W7.62mm
Changed lines of the file:
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@@
 			)
 		)
-		(property "Footprint" ""
+		(property "Footprint" "Package_DIP:DIP-14_W7.62mm"
 			(at 57.15 168.91 0)
 			(effects
@@
 			)
 		)
-		(property "Footprint" ""
+		(property "Footprint" "Capacitor_THT:C_Disc_D5.0mm_W2.5mm_P5.00mm"
 			(at 74.6252 63.5 0)
 			(effects
@@
 			)
 		)
-		(property "Footprint" ""
+		(property "Footprint" "Package_DIP:DIP-14_W7.62mm"
 			(at 34.29 182.88 0)
 			(effects
@@
 			)
 		)
-		(property "Footprint" ""
+		(property "Footprint" "Package_DIP:DIP-14_W7.62mm"
 			(at 29.21 36.83 0)
 			(effects
@@
 			)
 		)
-		(property "Footprint" ""
+		(property "Footprint" "Package_DIP:DIP-14_W7.62mm"
 			(at 55.88 182.88 0)
 			(effects
@@
 			)
 		)
-		(property "Footprint" ""
+		(property "Footprint" "Package_DIP:DIP-14_W7.62mm"
 			(at 77.47 168.91 0)
 			(effects
@@
 			)
 		)
-		(property "Footprint" ""
+		(property "Footprint" "Package_DIP:DIP-14_W7.62mm"
 			(at 151.13 88.9 0)
 			(effects
@@
 			)
 		)
-		(property "Footprint" ""
+		(property "Footprint" "Connector_PinHeader_2.54mm:PinHeader_1x03_P2.54mm_Vertical"
 			(at 64.77 31.75 0)
 			(effects
@@
 			)
 		)
-		(property "Footprint" ""
+		(property "Footprint" "Package_DIP:DIP-14_W7.62mm"
 			(at 34.29 168.91 0)
 			(effects
